Commit message: Made more stable thymio implementation

File: models/thymio/model.urdf (robot description, URDF)
Before this commit: robot thymio, 3 links, 2 joints
Links:
- added link caster; collision cylinder length=.001 radius=.01; visual sphere radius=.01
- link chassis: geometry collision mesh filename=package://models/thymio/meshes/gripper.dae scale=0.1 0.1 0.1; collision mesh filename=package://models/thymio/meshes/raspberry_case.dae scale=0.11 0.11 0.11
- link left_wheel: mass 0.01 -> None; geometry collision cylinder length=.015 radius=.021; visual cylinder length=.015 radius=.021
- link right_wheel: mass 0.01 -> None; geometry collision cylinder length=.015 radius=.021; visual cylinder length=.015 radius=.021
Joints:
- added joint caster_joint: type fixed, parent chassis, child caster, origin xyz=0 0 0 rpy=0 0 0
- joint left_wheel_hinge: limit lower=-2.8973 upper=2.8973 effort=12 velocity=2.6100 -> lower=-2.8973 upper=2.8973 effort=0.12 velocity=7; origin xyz=-0.027 0.05 -0.01 rpy=0 1.5707 1.5707 -> xyz=-0.027 0.0475 -0.01 rpy=0 1.5707 1.5707
- joint right_wheel_hinge: limit lower=-2.8973 upper=2.8973 effort=12 velocity=2.6100 -> lower=-2.8973 upper=2.8973 effort=0.12 velocity=7; origin xyz=-0.027 -0.05 -0.01 rpy=0 1.5707 1.5707 -> xyz=-0.027 -0.0475 -0.01 rpy=0 1.5707 1.5707

Commit message: New heading Sensor correct3ed, SoftReLU 300s 2rep exp

File: models/thymio/model.urdf (robot description, URDF)
Before this commit: robot thymio, 4 links, 3 joints
Links:
- link chassis: geometry collision mesh filename=package://models/thymio/meshes/raspberry_case.dae scale=0.11 0.11 0.11; collision mesh filename=package://models/thymio/meshes/thymio.dae

Commit message: Heterogenous swarm implementation (2 reservoirs)

File: models/thymio/model.urdf (robot description, URDF)
Before this commit: robot thymio, 4 links, 3 joints
Links:
- link caster: mass None -> 0.025; geometry collision cylinder length=.02 radius=.01; visual sphere radius=.01
- link chassis: mass 0.270 -> 0.170
- link left_wheel: mass None -> 0.075
- link right_wheel: mass None -> 0.075
Joints:
- joint left_wheel_hinge: origin xyz=-0.027 0.0475 -0.01 rpy=0 1.5707 1.5707 -> xyz=-0.027 0.0475 -0.01 rpy=-1.5707963267948966 0 0
- joint right_wheel_hinge: origin xyz=-0.027 -0.0475 -0.01 rpy=0 1.5707 1.5707 -> xyz=-0.027 -0.0475 -0.01 rpy=-1.5707963267948966 0 0

Commit message: Heterogenous swarm implementation (2 reservoirs), Stabalize thymio behaviour (.urdf)

File: models/thymio/model.urdf (robot description, URDF)
Before this commit: robot thymio, 4 links, 3 joints
Links:
- link chassis: mass 0.170 -> 0.230
